Commit message: Added synapses

File: body.urdf (robot description, URDF)
Before this commit: robot robot, 3 links, 2 joints
Joints:
- joint Torso_BackLeg: origin xyz=1 0 1 rpy=0 0 0 -> xyz=1 0 1.25 rpy=0 0 0
- joint Torso_FrontLeg: origin xyz=2 0 1 rpy=0 0 0 -> xyz=2 0 1.25 rpy=0 0 0

Commit message: Edited leg size

File: body.urdf (robot description, URDF)
Before this commit: robot robot, 3 links, 2 joints
Links:
- link BackLeg: geometry collision box size=0.2 1 0.2; visual box size=0.2 1 0.2
- link FrontLeg: geometry collision box size=0.2 1 0.2; visual box size=0.2 1 0.2
Joints:
- joint Torso_BackLeg: origin xyz=1 0 1.25 rpy=0 0 0 -> xyz=0 -0.5 1 rpy=0 0 0
- joint Torso_FrontLeg: origin xyz=2 0 1.25 rpy=0 0 0 -> xyz=0 0.5 1 rpy=0 0 0

Commit message: Added rollers

File: body.urdf (robot description, URDF)
Before this commit: robot robot, 9 links, 8 joints
Links:
- removed link BackLeg
- removed link BackLowerLeg
- removed link FrontLeg
- removed link FrontLowerLeg
- added link LeftArm, mass 1; collision box size=1 0.2 0.2; visual box size=1 0.2 0.2
- added link LeftRoller, mass 1; collision box size=1 0.2 0.2; visual box size=1 0.2 0.2
- added link RightArm, mass 1; collision box size=1 0.2 0.2; visual box size=1 0.2 0.2
- added link RightRoller, mass 1; collision box size=1 0.2 0.2; visual box size=1 0.2 0.2
- link LeftLeg: geometry collision box size=0.2 1 0.2; visual box size=0.2 1 0.2
- link RightLeg: geometry collision box size=0.2 1 0.2; visual box size=0.2 1 0.2
Joints:
- removed joint BackLeg_BackLowerLeg
- removed joint FrontLeg_FrontLowerLeg
- removed joint Torso_BackLeg
- removed joint Torso_FrontLeg
- added joint LeftLowerLeg_LeftRoller: type revolute, parent LeftLowerLeg, child LeftRoller, origin xyz=0.1 0 -0.9 rpy=0 0 0, axis 0 0 1, limit lower=-3.14159 upper=3.14159 effort=0.0 velocity=0.0
- added joint RightLowerLeg_RightRoller: type revolute, parent RightLowerLeg, child RightRoller, origin xyz=-0.1 0 -0.9 rpy=0 0 0, axis 0 0 1, limit lower=-3.14159 upper=3.14159 effort=0.0 velocity=0.0
- added joint Torso_LeftArm: type revolute, parent Torso, child LeftArm, origin xyz=-0.2 0.5 1.5 rpy=0 0 0, axis 0 1 0, limit lower=-3.14159 upper=3.14159 effort=0.0 velocity=0.0
- added joint Torso_RightArm: type revolute, parent Torso, child RightArm, origin xyz=0.2 0.5 1.5 rpy=0 0 0, axis 0 1 0, limit lower=-3.14159 upper=3.14159 effort=0.0 velocity=0.0
- joint LeftLeg_LeftLowerLeg: origin xyz=-1 0 0 rpy=0 0 0 -> xyz=0 -1 0 rpy=0 0 0
- joint RightLeg_RightLowerLeg: origin xyz=1 0 0 rpy=0 0 0 -> xyz=0 1 0 rpy=0 0 0
- joint Torso_LeftLeg: axis 0 1 0 -> 1 0 0; origin xyz=-0.5 0 1 rpy=0 0 0 -> xyz=-0.5 0 0.9 rpy=0 0 0
- joint Torso_RightLeg: axis 0 1 0 -> 1 0 0; origin xyz=0.5 0 1 rpy=0 0 0 -> xyz=0.5 0 0.9 rpy=0 0 0

Commit message: Fixed legs with rotating rollers

File: body.urdf (robot description, URDF)
Before this commit: robot robot, 9 links, 8 joints
Joints:
- joint LeftLeg_LeftLowerLeg: type revolute -> fixed
- joint LeftLowerLeg_LeftRoller: type revolute -> spherical
- joint RightLeg_RightLowerLeg: type revolute -> fixed
- joint RightLowerLeg_RightRoller: type revolute -> spherical
- joint Torso_LeftLeg: type revolute -> fixed
- joint Torso_RightLeg: type revolute -> fixed

Commit message: Rollers not rolling

File: body.urdf (robot description, URDF)
Before this commit: robot robot, 9 links, 8 joints
Joints:
- joint LeftLowerLeg_LeftRoller: origin xyz=0.1 0 -0.9 rpy=0 0 0 -> xyz=0.1 0 -1 rpy=0 0 0
- joint RightLowerLeg_RightRoller: origin xyz=-0.1 0 -0.9 rpy=0 0 0 -> xyz=-0.1 0 -1 rpy=0 0 0
- joint Torso_LeftLeg: axis 1 0 0 -> 0 0 1
- joint Torso_RightLeg: axis 1 0 0 -> 0 0 1

Commit message: Changed motor types

File: body.urdf (robot description, URDF)
Before this commit: robot robot, 9 links, 8 joints
Links:
- removed link LeftRoller
- removed link RightRoller
Joints:
- removed joint LeftLowerLeg_LeftRoller
- removed joint RightLowerLeg_RightRoller
- joint LeftLeg_LeftLowerLeg: type fixed -> planar
- joint RightLeg_RightLowerLeg: type fixed -> planar
- joint Torso_LeftLeg: axis 0 0 1 -> 1 0 0; type fixed -> revolute
- joint Torso_RightLeg: axis 0 0 1 -> 1 0 0; type fixed -> revolute

Commit message: Randomized links, haven't set up sensors yet

File: body.urdf (robot description, URDF)
Before this commit: robot robot, 9 links, 8 joints
Links:
- removed link BackLeg
- removed link BackLowerLeg
- removed link FrontLeg
- removed link FrontLowerLeg
- removed link LeftLeg
- removed link LeftLowerLeg
- removed link RightLeg
- removed link RightLowerLeg
- removed link Torso
- added link 0, mass 1; collision box size=1.6 0.1 0.9; visual box size=1.6 0.1 0.9
- added link 1, mass 1; collision box size=0.6 0.5 0.2; visual box size=0.6 0.5 0.2
- added link 2, mass 1; collision box size=0.7 0.2 1.2; visual box size=0.7 0.2 1.2
- added link 3, mass 1; collision box size=0.5 0.7 0.6; visual box size=0.5 0.7 0.6
- added link 4, mass 1; collision box size=0.7 0.9 0.3; visual box size=0.7 0.9 0.3
- added link 5, mass 1; collision box size=1.8 1.3 0.6; visual box size=1.8 1.3 0.6
- added link 6, mass 1; collision box size=1.5 1.1 1.9; visual box size=1.5 1.1 1.9
- added link 7, mass 1; collision box size=1.2 0.5 1.6; visual box size=1.2 0.5 1.6
Joints:
- removed joint BackLeg_BackLowerLeg
- removed joint FrontLeg_FrontLowerLeg
- removed joint LeftLeg_LeftLowerLeg
- removed joint RightLeg_RightLowerLeg
- removed joint Torso_BackLeg
- removed joint Torso_FrontLeg
- removed joint Torso_LeftLeg
- removed joint Torso_RightLeg
- added joint 0_1: type revolute, parent 0, child 1, origin xyz=1.6 0.1 1.9 rpy=0 0 0, axis 1 0 0, limit lower=-3.14159 upper=3.14159 effort=0.0 velocity=0.0
- added joint 1_2: type revolute, parent 1, child 2, origin xyz=0.6 0.5 0.2 rpy=0 0 0, axis 1 0 0, limit lower=-3.14159 upper=3.14159 effort=0.0 velocity=0.0
- added joint 2_3: type revolute, parent 2, child 3, origin xyz=0.7 0.2 1.2 rpy=0 0 0, axis 1 0 0, limit lower=-3.14159 upper=3.14159 effort=0.0 velocity=0.0
- added joint 3_4: type revolute, parent 3, child 4, origin xyz=0.5 0.7 0.6 rpy=0 0 0, axis 1 0 0, limit lower=-3.14159 upper=3.14159 effort=0.0 velocity=0.0
- added joint 4_5: type revolute, parent 4, child 5, origin xyz=0.7 0.9 0.3 rpy=0 0 0, axis 1 0 0, limit lower=-3.14159 upper=3.14159 effort=0.0 velocity=0.0
- added joint 5_6: type revolute, parent 5, child 6, origin xyz=1.8 1.3 0.6 rpy=0 0 0, axis 1 0 0, limit lower=-3.14159 upper=3.14159 effort=0.0 velocity=0.0
- added joint 6_7: type revolute, parent 6, child 7, origin xyz=1.5 1.1 1.9 rpy=0 0 0, axis 1 0 0, limit lower=-3.14159 upper=3.14159 effort=0.0 velocity=0.0

Commit message: Added color to sensors

File: body.urdf (robot description, URDF)
Before this commit: robot robot, 8 links, 7 joints
Links:
- added link 8, mass 1; collision box size=0.3 1.8 0.2; visual box size=0.3 1.8 0.2
- link 0: geometry collision box size=0.8 1.6 0.7; visual box size=0.8 1.6 0.7
- link 1: geometry collision box size=1.0 1.6 0.8; visual box size=1.0 1.6 0.8
- link 2: geometry collision box size=0.8 1.0 0.2; visual box size=0.8 1.0 0.2
- link 3: geometry collision box size=0.6 0.8 1.9; visual box size=0.6 0.8 1.9
- link 4: geometry collision box size=1.2 0.9 1.3; visual box size=1.2 0.9 1.3
- link 5: geometry collision box size=1.2 0.3 0.4; visual box size=1.2 0.3 0.4
- link 6: geometry collision box size=1.5 1.3 0.4; visual box size=1.5 1.3 0.4
- link 7: geometry collision box size=0.6 0.9 1.6; visual box size=0.6 0.9 1.6
Joints:
- added joint 7_8: type revolute, parent 7, child 8, origin xyz=0.6 0.9 1.6 rpy=0 0 0, axis 1 0 0, limit lower=-3.14159 upper=3.14159 effort=0.0 velocity=0.0
- joint 0_1: origin xyz=1.6 0.1 1.9 rpy=0 0 0 -> xyz=0.8 1.6 1.7 rpy=0 0 0
- joint 1_2: origin xyz=0.6 0.5 0.2 rpy=0 0 0 -> xyz=1.0 1.6 0.8 rpy=0 0 0
- joint 2_3: origin xyz=0.7 0.2 1.2 rpy=0 0 0 -> xyz=0.8 1.0 0.2 rpy=0 0 0
- joint 3_4: origin xyz=0.5 0.7 0.6 rpy=0 0 0 -> xyz=0.6 0.8 1.9 rpy=0 0 0
- joint 4_5: origin xyz=0.7 0.9 0.3 rpy=0 0 0 -> xyz=1.2 0.9 1.3 rpy=0 0 0
- joint 5_6: origin xyz=1.8 1.3 0.6 rpy=0 0 0 -> xyz=1.2 0.3 0.4 rpy=0 0 0
- joint 6_7: origin xyz=1.5 1.1 1.9 rpy=0 0 0 -> xyz=1.5 1.3 0.4 rpy=0 0 0

Commit message: Updated mutate function

File: body.urdf (robot description, URDF)
Before this commit: robot robot, 9 links, 8 joints
Links:
- removed link 2
- removed link 3
- removed link 4
- removed link 5
- removed link 6
- removed link 7
- removed link 8
- link 0: geometry collision box size=1.5 0.1 0.5; visual box size=1.5 0.1 0.5
- link 1: geometry collision box size=0.1 0.6 1.8; visual box size=0.1 0.6 1.8
Joints:
- removed joint 1_2
- removed joint 2_3
- removed joint 3_4
- removed joint 4_5
- removed joint 5_6
- removed joint 6_7
- removed joint 7_8
- joint 0_1: origin xyz=0.8 1.6 1.7 rpy=0 0 0 -> xyz=1.5 0.1 1.5 rpy=0 0 0

Commit message: Updated neuron indexing

File: body.urdf (robot description, URDF)
Before this commit: robot robot, 2 links, 1 joints
Links:
- added link 2, mass 1; collision box size=0.6 0.8 0.2; visual box size=0.6 0.8 0.2
- added link 3, mass 1; collision box size=0.5 1.9 1.6; visual box size=0.5 1.9 1.6
- link 0: geometry collision box size=1.6 1.0 1.5; visual box size=1.6 1.0 1.5
- link 1: geometry collision box size=0.2 0.6 0.3; visual box size=0.2 0.6 0.3
Joints:
- added joint 1_2: type revolute, parent 1, child 2, origin xyz=0.2 0.6 0.3 rpy=0 0 0, axis 1 0 0, limit lower=-3.14159 upper=3.14159 effort=0.0 velocity=0.0
- added joint 2_3: type revolute, parent 2, child 3, origin xyz=0.6 0.8 0.2 rpy=0 0 0, axis 1 0 0, limit lower=-3.14159 upper=3.14159 effort=0.0 velocity=0.0
- joint 0_1: origin xyz=1.5 0.1 1.5 rpy=0 0 0 -> xyz=1.6 1.0 2.5 rpy=0 0 0

Commit message: Fixed colors and updated neuron indexing

File: body.urdf (robot description, URDF)
Before this commit: robot robot, 4 links, 3 joints
Links:
- removed link 2
- removed link 3
- link 0: geometry collision box size=1.7 0.4 1.3; visual box size=1.7 0.4 1.3
- link 1: geometry collision box size=0.2 1.8 1.1; visual box size=0.2 1.8 1.1
Joints:
- removed joint 1_2
- removed joint 2_3
- joint 0_1: origin xyz=1.6 1.0 2.5 rpy=0 0 0 -> xyz=0.85 0.2 1.15 rpy=0 0 0

Commit message: Removed sidebars from sim

File: body.urdf (robot description, URDF)
Before this commit: robot robot, 2 links, 1 joints
Links:
- added link 2, mass 1; collision box size=0.7 1.3 1.0; visual box size=0.7 1.3 1.0
- added link 3, mass 1; collision box size=0.6 1.7 1.9; visual box size=0.6 1.7 1.9
- link 0: geometry collision box size=0.4 1.2 1.3; visual box size=0.4 1.2 1.3
- link 1: geometry collision box size=0.6 0.5 1.8; visual box size=0.6 0.5 1.8
Joints:
- added joint 1_2: type revolute, parent 1, child 2, origin xyz=0.6 0.5 1.8 rpy=0 0 0, axis 1 0 0, limit lower=-3.14159 upper=3.14159 effort=0.0 velocity=0.0
- added joint 2_3: type revolute, parent 2, child 3, origin xyz=0.7 1.3 1.0 rpy=0 0 0, axis 1 0 0, limit lower=-3.14159 upper=3.14159 effort=0.0 velocity=0.0
- joint 0_1: origin xyz=0.85 0.2 1.15 rpy=0 0 0 -> xyz=0.4 1.2 1.3 rpy=0 0 0

Commit message: Set snake on the ground

File: body.urdf (robot description, URDF)
Before this commit: robot robot, 4 links, 3 joints
Links:
- removed link 2
- removed link 3
- link 0: geometry collision box size=1.4 1.6 0.7; visual box size=1.4 1.6 0.7
- link 1: geometry collision box size=1.9 0.6 1.6; visual box size=1.9 0.6 1.6
Joints:
- removed joint 1_2
- removed joint 2_3
- joint 0_1: origin xyz=0.4 1.2 1.3 rpy=0 0 0 -> xyz=1.4 0 1 rpy=0 0 0

Commit message: Changed motor values, fixed nonetype error

File: body.urdf (robot description, URDF)
Before this commit: robot robot, 2 links, 1 joints
Links:
- added link 2, mass 1; collision box size=1.4 0.6 0.7; visual box size=1.4 0.6 0.7
- added link 3, mass 1; collision box size=0.7 0.5 1.3; visual box size=0.7 0.5 1.3
- added link 4, mass 1; collision box size=0.5 1.7 1.3; visual box size=0.5 1.7 1.3
- added link 5, mass 1; collision box size=1.0 0.8 1.5; visual box size=1.0 0.8 1.5
- link 0: geometry collision box size=0.6 1.6 0.4; visual box size=0.6 1.6 0.4
- link 1: geometry collision box size=0.9 1.7 1.5; visual box size=0.9 1.7 1.5
Joints:
- added joint 1_2: type revolute, parent 1, child 2, origin xyz=0.9 0 0 rpy=0 0 0, axis 1 1 0, limit lower=-3.14159 upper=3.14159 effort=0.0 velocity=0.0
- added joint 2_3: type revolute, parent 2, child 3, origin xyz=1.4 0 0 rpy=0 0 0, axis 1 1 0, limit lower=-3.14159 upper=3.14159 effort=0.0 velocity=0.0
- added joint 3_4: type revolute, parent 3, child 4, origin xyz=0.7 0 0 rpy=0 0 0, axis 1 1 0, limit lower=-3.14159 upper=3.14159 effort=0.0 velocity=0.0
- added joint 4_5: type revolute, parent 4, child 5, origin xyz=0.5 0 0 rpy=0 0 0, axis 1 1 0, limit lower=-3.14159 upper=3.14159 effort=0.0 velocity=0.0
- joint 0_1: axis 1 0 0 -> 1 1 0; origin xyz=1.4 0 1 rpy=0 0 0 -> xyz=0.6 0 1 rpy=0 0 0

Commit message: Added min and max links to constants

File: body.urdf (robot description, URDF)
Before this commit: robot robot, 6 links, 5 joints
Links:
- added link 6, mass 1; collision box size=1.8 0.7 0.6; visual box size=1.8 0.7 0.6
- added link 7, mass 1; collision box size=1.8 0.7 0.5; visual box size=1.8 0.7 0.5
- link 0: geometry collision box size=0.2 1.8 1.3; visual box size=0.2 1.8 1.3
- link 1: geometry collision box size=1.6 0.1 1.7; visual box size=1.6 0.1 1.7
- link 2: geometry collision box size=0.6 0.1 1.1; visual box size=0.6 0.1 1.1
- link 3: geometry collision box size=0.9 0.5 0.2; visual box size=0.9 0.5 0.2
- link 4: geometry collision box size=0.9 0.2 0.6; visual box size=0.9 0.2 0.6
- link 5: geometry collision box size=1.8 1.4 0.4; visual box size=1.8 1.4 0.4
Joints:
- added joint 5_6: type revolute, parent 5, child 6, origin xyz=1.8 0 0 rpy=0 0 0, axis 1 1 0, limit lower=-3.14159 upper=3.14159 effort=0.0 velocity=0.0
- added joint 6_7: type revolute, parent 6, child 7, origin xyz=1.8 0 0 rpy=0 0 0, axis 1 1 0, limit lower=-3.14159 upper=3.14159 effort=0.0 velocity=0.0
- joint 0_1: origin xyz=0.6 0 1 rpy=0 0 0 -> xyz=0.2 0 1 rpy=0 0 0
- joint 1_2: origin xyz=0.9 0 0 rpy=0 0 0 -> xyz=1.6 0 0 rpy=0 0 0
- joint 2_3: origin xyz=1.4 0 0 rpy=0 0 0 -> xyz=0.6 0 0 rpy=0 0 0
- joint 3_4: origin xyz=0.7 0 0 rpy=0 0 0 -> xyz=0.9 0 0 rpy=0 0 0
- joint 4_5: origin xyz=0.5 0 0 rpy=0 0 0 -> xyz=0.9 0 0 rpy=0 0 0

Commit message: Changed fitness function and motor ranges

File: body.urdf (robot description, URDF)
Before this commit: robot robot, 8 links, 7 joints
Links:
- removed link 6
- removed link 7
- link 0: geometry collision box size=0.5 1.3 1.2; visual box size=0.5 1.3 1.2
- link 1: geometry collision box size=0.2 0.6 1.7; visual box size=0.2 0.6 1.7
- link 2: geometry collision box size=1.8 0.3 0.4; visual box size=1.8 0.3 0.4
- link 3: geometry collision box size=1.5 1.2 0.2; visual box size=1.5 1.2 0.2
- link 4: geometry collision box size=1.1 1.0 0.7; visual box size=1.1 1.0 0.7
- link 5: geometry collision box size=0.1 1.3 1.5; visual box size=0.1 1.3 1.5
Joints:
- removed joint 5_6
- removed joint 6_7
- joint 0_1: origin xyz=0.2 0 1 rpy=0 0 0 -> xyz=0.5 0 1 rpy=0 0 0
- joint 1_2: origin xyz=1.6 0 0 rpy=0 0 0 -> xyz=0.2 0 0 rpy=0 0 0
- joint 2_3: origin xyz=0.6 0 0 rpy=0 0 0 -> xyz=1.8 0 0 rpy=0 0 0
- joint 3_4: origin xyz=0.9 0 0 rpy=0 0 0 -> xyz=1.5 0 0 rpy=0 0 0
- joint 4_5: origin xyz=0.9 0 0 rpy=0 0 0 -> xyz=1.1 0 0 rpy=0 0 0

Commit message: Recursively creating link limbs

File: body.urdf (robot description, URDF)
Before this commit: robot robot, 6 links, 5 joints
Links:
- added link 6, mass 1; collision box size=0.4 1.9 1.1; visual box size=0.4 1.9 1.1
- added link 7, mass 1; collision box size=0.5 0.1 1.5; visual box size=0.5 0.1 1.5
- link 0: geometry collision box size=0.4 1.8 1.4; visual box size=0.4 1.8 1.4
- link 1: geometry collision box size=0.1 0.9 1.7; visual box size=0.1 0.9 1.7
- link 2: geometry collision box size=0.7 1.6 1.3; visual box size=0.7 1.6 1.3
- link 3: geometry collision box size=0.6 0.1 0.4; visual box size=0.6 0.1 0.4
- link 4: geometry collision box size=0.1 1.2 1.0; visual box size=0.1 1.2 1.0
- link 5: geometry collision box size=1.6 1.9 0.5; visual box size=1.6 1.9 0.5
Joints:
- added joint 5_6: type revolute, parent 5, child 6, origin xyz=1.6 0 0 rpy=0 0 0, axis 1 1 0, limit lower=-3.14159 upper=3.14159 effort=0.0 velocity=0.0
- added joint 6_7: type revolute, parent 6, child 7, origin xyz=0.4 0 0 rpy=0 0 0, axis 1 1 0, limit lower=-3.14159 upper=3.14159 effort=0.0 velocity=0.0
- joint 0_1: origin xyz=0.5 0 1 rpy=0 0 0 -> xyz=0.4 0 1 rpy=0 0 0
- joint 1_2: origin xyz=0.2 0 0 rpy=0 0 0 -> xyz=0.1 0 0 rpy=0 0 0
- joint 2_3: origin xyz=1.8 0 0 rpy=0 0 0 -> xyz=0.7 0 0 rpy=0 0 0
- joint 3_4: origin xyz=1.5 0 0 rpy=0 0 0 -> xyz=0.6 0 0 rpy=0 0 0
- joint 4_5: origin xyz=1.1 0 0 rpy=0 0 0 -> xyz=0.1 0 0 rpy=0 0 0

Commit message: Updated generate brain

File: body.urdf (robot description, URDF)
Before this commit: robot robot, 8 links, 7 joints
Links:
- added link 10, mass 1; collision box size=0.4 0.2 1.4; visual box size=0.4 0.2 1.4
- added link 8, mass 1; collision box size=0.5 1.5 1.9; visual box size=0.5 1.5 1.9
- added link 9, mass 1; collision box size=0.5 0.3 1.4; visual box size=0.5 0.3 1.4
- link 0: geometry collision box size=0.4 0.9 1.8; visual box size=0.4 0.9 1.8
- link 1: geometry collision box size=0.2 1.5 1.1; visual box size=0.2 1.5 1.1
- link 2: geometry collision box size=0.9 1.4 0.6; visual box size=0.9 1.4 0.6
- link 3: geometry collision box size=0.9 1.5 0.6; visual box size=0.9 1.5 0.6
- link 4: geometry collision box size=1.2 1.9 0.3; visual box size=1.2 1.9 0.3
- link 5: geometry collision box size=1.1 1.6 0.3; visual box size=1.1 1.6 0.3
- link 6: geometry collision box size=1.7 1.5 0.2; visual box size=1.7 1.5 0.2
- link 7: geometry collision box size=0.9 1.6 1.9; visual box size=0.9 1.6 1.9
Joints:
- added joint 7_8: type revolute, parent 7, child 8, origin xyz=-0.45 0 0.95 rpy=0 0 0, axis 1 1 0, limit lower=-3.14159 upper=3.14159 effort=0.0 velocity=0.0
- added joint 8_9: type revolute, parent 8, child 9, origin xyz=-0.5 0 0 rpy=0 0 0, axis 1 1 0, limit lower=-3.14159 upper=3.14159 effort=0.0 velocity=0.0
- joint 0_1: origin xyz=0.4 0 1 rpy=0 0 0 -> xyz=0.2 -0.45 1 rpy=0 0 0
- joint 1_2: origin xyz=0.1 0 0 rpy=0 0 0 -> xyz=0 -1.5 0 rpy=0 0 0
- joint 2_3: origin xyz=0.7 0 0 rpy=0 0 0 -> xyz=0 -0.7 0.3 rpy=0 0 0
- joint 3_4: origin xyz=0.6 0 0 rpy=0 0 0 -> xyz=0 0 0.6 rpy=0 0 0
- joint 4_5: origin xyz=0.1 0 0 rpy=0 0 0 -> xyz=0 -0.95 0.15 rpy=0 0 0
- joint 5_6: origin xyz=1.6 0 0 rpy=0 0 0 -> xyz=-0.55 -0.8 0 rpy=0 0 0
- joint 6_7: origin xyz=0.4 0 0 rpy=0 0 0 -> xyz=-0.85 0 0.1 rpy=0 0 0

Commit message: Running solution for only one iteration, joints not properly connected

File: body.urdf (robot description, URDF)
Before this commit: robot robot, 11 links, 9 joints
Links:
- removed link 10
- removed link 3
- removed link 4
- removed link 5
- removed link 6
- removed link 7
- removed link 8
- removed link 9
- link 0: geometry collision box size=1.3 1.0 1.7; visual box size=1.3 1.0 1.7
- link 1: geometry collision box size=0.8 1.6 0.7; visual box size=0.8 1.6 0.7
- link 2: geometry collision box size=1.6 1.7 0.8; visual box size=1.6 1.7 0.8
Joints:
- removed joint 2_3
- removed joint 3_4
- removed joint 4_5
- removed joint 5_6
- removed joint 6_7
- removed joint 7_8
- removed joint 8_9
- joint 0_1: origin xyz=0.2 -0.45 1 rpy=0 0 0 -> xyz=1.3 0 1 rpy=0 0 0
- joint 1_2: origin xyz=0 -1.5 0 rpy=0 0 0 -> xyz=0.4 -0.8 0 rpy=0 0 0

Commit message: 3D creatures are being generated. Need to track sizes so blocks do not overlap

File: body.urdf (robot description, URDF)
Before this commit: robot robot, 3 links, 2 joints
Links:
- added link 3, mass 1; collision box size=1.0 0.4 1.7; visual box size=1.0 0.4 1.7
- added link 4, mass 1; collision box size=0.8 0.6 0.4; visual box size=0.8 0.6 0.4
- added link 5, mass 1; collision box size=1.3 1.1 0.2; visual box size=1.3 1.1 0.2
- added link 6, mass 1; collision box size=0.2 0.8 1.1; visual box size=0.2 0.8 1.1
- added link 7, mass 1; collision box size=1.8 0.6 1.9; visual box size=1.8 0.6 1.9
- added link 8, mass 1; collision box size=1.9 1.7 1.8; visual box size=1.9 1.7 1.8
- link 0: geometry collision box size=1.8 0.9 0.6; visual box size=1.8 0.9 0.6
- link 1: geometry collision box size=0.5 0.6 1.3; visual box size=0.5 0.6 1.3
- link 2: geometry collision box size=1.0 1.5 1.7; visual box size=1.0 1.5 1.7
Joints:
- added joint 2_3: type revolute, parent 2, child 3, origin xyz=-1.0 0 0 rpy=0 0 0, axis 1 1 0, limit lower=-3.14159 upper=3.14159 effort=0.0 velocity=0.0
- added joint 3_4: type revolute, parent 3, child 4, origin xyz=-0.5 0 0.85 rpy=0 0 0, axis 1 1 0, limit lower=-3.14159 upper=3.14159 effort=0.0 velocity=0.0
- added joint 4_5: type revolute, parent 4, child 5, origin xyz=-0.4 0 0.2 rpy=0 0 0, axis 1 1 0, limit lower=-3.14159 upper=3.14159 effort=0.0 velocity=0.0
- added joint 5_6: type revolute, parent 5, child 6, origin xyz=-0.65 0.55 0 rpy=0 0 0, axis 1 1 0, limit lower=-3.14159 upper=3.14159 effort=0.0 velocity=0.0
- added joint 6_7: type revolute, parent 6, child 7, origin xyz=0 0.8 0 rpy=0 0 0, axis 1 1 0, limit lower=-3.14159 upper=3.14159 effort=0.0 velocity=0.0
- added joint 7_8: type revolute, parent 7, child 8, origin xyz=0 0.6 0 rpy=0 0 0, axis 1 1 0, limit lower=-3.14159 upper=3.14159 effort=0.0 velocity=0.0
- joint 0_1: origin xyz=1.3 0 1 rpy=0 0 0 -> xyz=0 0.45 1.3 rpy=0 0 0
- joint 1_2: origin xyz=0.4 -0.8 0 rpy=0 0 0 -> xyz=-0.25 0.3 0 rpy=0 0 0

Commit message: Changed self.lastAbsolutePos into a dictionary of link positions, preparing to add multiple links to each link face

File: body.urdf (robot description, URDF)
Before this commit: robot robot, 9 links, 8 joints
Links:
- link 0: geometry collision box size=0.3 1.4 0.1; visual box size=0.3 1.4 0.1
- link 1: geometry collision box size=0.4 1.9 0.7; visual box size=0.4 1.9 0.7
- link 2: geometry collision box size=1.7 0.7 1.2; visual box size=1.7 0.7 1.2
- link 3: geometry collision box size=1.9 0.5 1.2; visual box size=1.9 0.5 1.2
- link 4: geometry collision box size=0.6 1.0 1.2; visual box size=0.6 1.0 1.2
- link 5: geometry collision box size=0.3 1.1 0.1; visual box size=0.3 1.1 0.1
- link 6: geometry collision box size=1.8 1.5 0.9; visual box size=1.8 1.5 0.9
- link 7: geometry collision box size=0.7 1.7 1.5; visual box size=0.7 1.7 1.5
- link 8: geometry collision box size=1.7 0.8 0.9; visual box size=1.7 0.8 0.9
Joints:
- joint 0_1: origin xyz=0 0 1.5 rpy=0 0 0 -> xyz=0.15 0 1 rpy=0 0 0
- joint 1_2: origin xyz=-0.7 0 0.4 rpy=0 0 0 -> xyz=0.2 0.95 0 rpy=0 0 0
- joint 2_3: origin xyz=-0.2 0 0.5 rpy=0 0 0 -> xyz=0 0.7 0 rpy=0 0 0
- joint 3_4: origin xyz=0 0 1.7 rpy=0 0 0 -> xyz=0 0.5 0 rpy=0 0 0
- joint 4_5: origin xyz=0 -0.45 0.85 rpy=0 0 0 -> xyz=0 1.0 0 rpy=0 0 0
- joint 5_6: origin xyz=-0.1 -0.65 0 rpy=0 0 0 -> xyz=0 0.55 0.05 rpy=0 0 0
- joint 6_7: origin xyz=-1.5 0 0 rpy=0 0 0 -> xyz=0.9 0 0.45 rpy=0 0 0
- joint 7_8: origin xyz=-1.3 0 0 rpy=0 0 0 -> xyz=0.7 0 0 rpy=0 0 0
