Commit message: Restructured intersection check

File: body.urdf (robot description, URDF)
Before this commit: robot robot, 9 links, 8 joints
Links:
- link 0: geometry collision box size=1.9 1.3 1.1; visual box size=1.9 1.3 1.1
- link 1: geometry collision box size=1.8 1.9 1.4; visual box size=1.8 1.9 1.4
- link 2: geometry collision box size=0.6 0.3 1.4; visual box size=0.6 0.3 1.4
- link 3: geometry collision box size=0.6 1.3 1.1; visual box size=0.6 1.3 1.1
- link 4: geometry collision box size=0.6 0.8 1.1; visual box size=0.6 0.8 1.1
- link 5: geometry collision box size=1.8 0.7 1.4; visual box size=1.8 0.7 1.4
- link 6: geometry collision box size=0.3 0.5 1.8; visual box size=0.3 0.5 1.8
- link 7: geometry collision box size=0.5 0.8 0.9; visual box size=0.5 0.8 0.9
- link 8: geometry collision box size=1.3 1.1 1.5; visual box size=1.3 1.1 1.5
Joints:
- joint 0_1: origin xyz=0.15 0 1 rpy=0 0 0 -> xyz=0.95 0 1 rpy=0 0 0
- joint 1_2: origin xyz=0.2 0.95 0 rpy=0 0 0 -> xyz=0.9 0.95 0 rpy=0 0 0
- joint 2_3: origin xyz=0 0.7 0 rpy=0 0 0 -> xyz=0 0.3 0 rpy=0 0 0
- joint 3_4: origin xyz=0 0.5 0 rpy=0 0 0 -> xyz=0.3 0.65 0 rpy=0 0 0
- joint 4_5: origin xyz=0 1.0 0 rpy=0 0 0 -> xyz=0.6 0 0 rpy=0 0 0
- joint 5_6: origin xyz=0 0.55 0.05 rpy=0 0 0 -> xyz=0.9 0 0.7 rpy=0 0 0
- joint 6_7: origin xyz=0.9 0 0.45 rpy=0 0 0 -> xyz=0 0.25 0.9 rpy=0 0 0
- joint 7_8: origin xyz=0.7 0 0 rpy=0 0 0 -> xyz=0.25 0.4 0 rpy=0 0 0

Commit message: Changed name of depth

File: body.urdf (robot description, URDF)
Before this commit: robot robot, 9 links, 8 joints
Links:
- removed link 6
- removed link 7
- removed link 8
- link 0: geometry collision box size=1.3 0.1 1.2; visual box size=1.3 0.1 1.2
- link 1: geometry collision box size=4.5 1.0 0.5; visual box size=4.5 1.0 0.5
- link 2: geometry collision box size=3.5 4.0 2.0; visual box size=3.5 4.0 2.0
- link 3: geometry collision box size=2.5 1.0 0.5; visual box size=2.5 1.0 0.5
- link 4: geometry collision box size=0.15000000000000585 1.0000000000000027 1.5; visual box size=0.15000000000000585 1.0000000000000027 1.5
- link 5: geometry collision box size=1.0 4.0 3.0; visual box size=1.0 4.0 3.0
Joints:
- removed joint 5_6
- removed joint 6_7
- removed joint 7_8
- joint 0_1: origin xyz=0.95 0 1 rpy=0 0 0 -> xyz=0 -0.05 1 rpy=0 0 0
- joint 1_2: origin xyz=0.9 0.95 0 rpy=0 0 0 -> xyz=0 -1.0 0 rpy=0 0 0
- joint 2_3: origin xyz=0 0.3 0 rpy=0 0 0 -> xyz=0 -4.0 0 rpy=0 0 0
- joint 3_4: origin xyz=0.3 0.65 0 rpy=0 0 0 -> xyz=0 -0.5 0.25 rpy=0 0 0
- joint 4_5: origin xyz=0.6 0 0 rpy=0 0 0 -> xyz=0 0 1.5 rpy=0 0 0

Commit message: About to change link space checking

File: body.urdf (robot description, URDF)
Before this commit: robot robot, 6 links, 5 joints
Links:
- link 0: geometry collision box size=0.2 1.0 0.5; visual box size=0.2 1.0 0.5
- link 1: geometry collision box size=4.0 2.0 1.0; visual box size=4.0 2.0 1.0
- link 2: geometry collision box size=4.0 4.5 1.5; visual box size=4.0 4.5 1.5
- link 3: geometry collision box size=3.5 0.5 2.0; visual box size=3.5 0.5 2.0
- link 4: geometry collision box size=1.0 2.5 4.0; visual box size=1.0 2.5 4.0
- link 5: geometry collision box size=2.5 3.0 3.5; visual box size=2.5 3.0 3.5
Joints:
- joint 0_1: origin xyz=0 -0.05 1 rpy=0 0 0 -> xyz=-0.1 0 1 rpy=0 0 0
- joint 1_2: origin xyz=0 -1.0 0 rpy=0 0 0 -> xyz=-2.0 -1.0 0 rpy=0 0 0
- joint 2_3: origin xyz=0 -4.0 0 rpy=0 0 0 -> xyz=0 -4.5 0 rpy=0 0 0
- joint 3_4: origin xyz=0 -0.5 0.25 rpy=0 0 0 -> xyz=-4.0 0 0 rpy=0 0 0
- joint 4_5: origin xyz=0 0 1.5 rpy=0 0 0 -> xyz=-1.0 0 0 rpy=0 0 0

Commit message: Fixed link spacing

File: body.urdf (robot description, URDF)
Before this commit: robot robot, 6 links, 5 joints
Links:
- added link 10, mass 1; collision box size=1.5 4.0 0.5; visual box size=1.5 4.0 0.5
- added link 11, mass 1; collision box size=4.5 3.5 3.0; visual box size=4.5 3.5 3.0
- added link 12, mass 1; collision box size=1.5 1.0 2.5; visual box size=1.5 1.0 2.5
- added link 13, mass 1; collision box size=2.0 1.0 2.5; visual box size=2.0 1.0 2.5
- added link 14, mass 1; collision box size=2.0 3.5 2.5; visual box size=2.0 3.5 2.5
- added link 15, mass 1; collision box size=2.0 3.5 4.5; visual box size=2.0 3.5 4.5
- added link 16, mass 1; collision box size=1.0 2.0 3.0; visual box size=1.0 2.0 3.0
- added link 6, mass 1; collision box size=3.0 2.0 2.5; visual box size=3.0 2.0 2.5
- added link 7, mass 1; collision box size=2.5 4.0 3.0; visual box size=2.5 4.0 3.0
- added link 8, mass 1; collision box size=4.5 1.5 2.0; visual box size=4.5 1.5 2.0
- added link 9, mass 1; collision box size=2.5 3.0 4.5; visual box size=2.5 3.0 4.5
- link 0: geometry collision box size=0.8 0.6 1.7; visual box size=0.8 0.6 1.7
- link 1: geometry collision box size=4.5 1.0 3.0; visual box size=4.5 1.0 3.0
- link 2: geometry collision box size=3.0 1.0 1.5; visual box size=3.0 1.0 1.5
- link 3: geometry collision box size=1.0 1.5 0.5; visual box size=1.0 1.5 0.5
- link 4: geometry collision box size=2.0 3.0 4.5; visual box size=2.0 3.0 4.5
- link 5: geometry collision box size=0.5 4.5 2.5; visual box size=0.5 4.5 2.5
Joints:
- removed joint 4_5
- added joint 11_12: type revolute, parent 11, child 12, origin xyz=0 3.5 0 rpy=0 0 0, axis 1 1 0, limit lower=-3.14159 upper=3.14159 effort=0.0 velocity=0.0
- added joint 12_13: type revolute, parent 12, child 13, origin xyz=0 1.0 0 rpy=0 0 0, axis 1 1 0, limit lower=-3.14159 upper=3.14159 effort=0.0 velocity=0.0
- added joint 14_15: type revolute, parent 14, child 15, origin xyz=0 0 2.5 rpy=0 0 0, axis 1 1 0, limit lower=-3.14159 upper=3.14159 effort=0.0 velocity=0.0
- added joint 15_16: type revolute, parent 15, child 16, origin xyz=0 0 4.5 rpy=0 0 0, axis 1 1 0, limit lower=-3.14159 upper=3.14159 effort=0.0 velocity=0.0
- added joint 1_11: type revolute, parent 1, child 11, origin xyz=0 0.5 1.5 rpy=0 0 0, axis 1 1 0, limit lower=-3.14159 upper=3.14159 effort=0.0 velocity=0.0
- added joint 1_14: type revolute, parent 1, child 14, origin xyz=0 0 3.0 rpy=0 0 0, axis 1 1 0, limit lower=-3.14159 upper=3.14159 effort=0.0 velocity=0.0
- added joint 1_5: type revolute, parent 1, child 5, origin xyz=-2.25 0 1.5 rpy=0 0 0, axis 1 1 0, limit lower=-3.14159 upper=3.14159 effort=0.0 velocity=0.0
- added joint 1_8: type revolute, parent 1, child 8, origin xyz=2.25 0 1.5 rpy=0 0 0, axis 1 1 0, limit lower=-3.14159 upper=3.14159 effort=0.0 velocity=0.0
- added joint 5_6: type revolute, parent 5, child 6, origin xyz=-0.5 0 0 rpy=0 0 0, axis 1 1 0, limit lower=-3.14159 upper=3.14159 effort=0.0 velocity=0.0
- added joint 6_7: type revolute, parent 6, child 7, origin xyz=-3.0 0 0 rpy=0 0 0, axis 1 1 0, limit lower=-3.14159 upper=3.14159 effort=0.0 velocity=0.0
- added joint 8_9: type revolute, parent 8, child 9, origin xyz=4.5 0 0 rpy=0 0 0, axis 1 1 0, limit lower=-3.14159 upper=3.14159 effort=0.0 velocity=0.0
- added joint 9_10: type revolute, parent 9, child 10, origin xyz=2.5 0 0 rpy=0 0 0, axis 1 1 0, limit lower=-3.14159 upper=3.14159 effort=0.0 velocity=0.0
- joint 0_1: origin xyz=-0.1 0 1 rpy=0 0 0 -> xyz=0 0 1.85 rpy=0 0 0
- joint 1_2: origin xyz=-2.0 -1.0 0 rpy=0 0 0 -> xyz=0 -0.5 1.5 rpy=0 0 0
- joint 2_3: origin xyz=0 -4.5 0 rpy=0 0 0 -> xyz=0 -1.0 0 rpy=0 0 0
- joint 3_4: origin xyz=-4.0 0 0 rpy=0 0 0 -> xyz=0 -1.5 0 rpy=0 0 0

Commit message: Starting to create new body files for each generation. Keep in mind that Create_Body is called each generation. Need body plan to execute in Create_Body that is predetermined

File: body.urdf (robot description, URDF)
Before this commit: robot robot, 17 links, 16 joints
Links:
- removed link 10
- removed link 11
- removed link 12
- removed link 13
- removed link 14
- removed link 15
- removed link 16
- removed link 8
- removed link 9
- link 0: geometry collision box size=1.0 0.7 1.6; visual box size=1.0 0.7 1.6
- link 1: geometry collision box size=3.5 3.0 1.5; visual box size=3.5 3.0 1.5
- link 2: geometry collision box size=1.0 4.5 3.5; visual box size=1.0 4.5 3.5
- link 3: geometry collision box size=2.5 3.0 1.5; visual box size=2.5 3.0 1.5
- link 4: geometry collision box size=2.0 1.0 4.5; visual box size=2.0 1.0 4.5
- link 5: geometry collision box size=3.0 0.5 2.5; visual box size=3.0 0.5 2.5
- link 6: geometry collision box size=1.0 0.5 3.0; visual box size=1.0 0.5 3.0
- link 7: geometry collision box size=3.0 2.0 0.5; visual box size=3.0 2.0 0.5
Joints:
- removed joint 11_12
- removed joint 12_13
- removed joint 14_15
- removed joint 15_16
- removed joint 1_11
- removed joint 1_14
- removed joint 1_8
- removed joint 8_9
- removed joint 9_10
- joint 0_1: origin xyz=0 0 1.85 rpy=0 0 0 -> xyz=0.5 0 1 rpy=0 0 0
- joint 1_2: origin xyz=0 -0.5 1.5 rpy=0 0 0 -> xyz=3.5 0 0 rpy=0 0 0
- joint 1_5: origin xyz=-2.25 0 1.5 rpy=0 0 0 -> xyz=1.75 0 0.75 rpy=0 0 0
- joint 2_3: origin xyz=0 -1.0 0 rpy=0 0 0 -> xyz=0.5 -2.25 0 rpy=0 0 0
- joint 3_4: origin xyz=0 -1.5 0 rpy=0 0 0 -> xyz=0 -3.0 0 rpy=0 0 0
- joint 5_6: origin xyz=-0.5 0 0 rpy=0 0 0 -> xyz=0 0 2.5 rpy=0 0 0
- joint 6_7: origin xyz=-3.0 0 0 rpy=0 0 0 -> xyz=0 0.25 1.5 rpy=0 0 0

Commit message: Changed to body plan system. Updating neuron generation methods

File: body.urdf (robot description, URDF)
Before this commit: robot robot, 8 links, 7 joints
Links:
- link 0: geometry collision box size=0.2 0.5 1.6; visual box size=0.2 0.5 1.6
- link 1: geometry collision box size=1.0 3.5 3.0; visual box size=1.0 3.5 3.0
- link 2: geometry collision box size=0.5 1.5 3.0; visual box size=0.5 1.5 3.0
- link 3: geometry collision box size=1.0 4.5 2.0; visual box size=1.0 4.5 2.0
- link 4: geometry collision box size=4.5 3.5 3.0; visual box size=4.5 3.5 3.0
- link 5: geometry collision box size=1.5 2.5 2.0; visual box size=1.5 2.5 2.0
- link 6: geometry collision box size=2.0 1.0 3.5; visual box size=2.0 1.0 3.5
- link 7: geometry collision box size=3.0 4.5 3.5; visual box size=3.0 4.5 3.5
Joints:
- joint 0_1: origin xyz=0.5 0 1 rpy=0 0 0 -> xyz=0.1 0 1 rpy=0 0 0
- joint 1_2: origin xyz=3.5 0 0 rpy=0 0 0 -> xyz=1.0 0 0 rpy=0 0 0
- joint 1_5: origin xyz=1.75 0 0.75 rpy=0 0 0 -> xyz=0.5 1.75 0 rpy=0 0 0
- joint 2_3: origin xyz=0.5 -2.25 0 rpy=0 0 0 -> xyz=0.5 0 0 rpy=0 0 0
- joint 3_4: origin xyz=0 -3.0 0 rpy=0 0 0 -> xyz=1.0 0 0 rpy=0 0 0
- joint 5_6: origin xyz=0 0 2.5 rpy=0 0 0 -> xyz=0 2.5 0 rpy=0 0 0
- joint 6_7: origin xyz=0 0.25 1.5 rpy=0 0 0 -> xyz=0 0.5 1.75 rpy=0 0 0

Commit message: Fixed brain and body plan generation

File: body.urdf (robot description, URDF)
Before this commit: robot robot, 8 links, 7 joints
Links:
- removed link 3
- removed link 4
- removed link 5
- removed link 6
- removed link 7
- link 0: geometry collision box size=1.9 1.2 0.7; visual box size=1.9 1.2 0.7
- link 1: geometry collision box size=4.5 4.0 3.0; visual box size=4.5 4.0 3.0
- link 2: geometry collision box size=0.5 2.0 4.5; visual box size=0.5 2.0 4.5
Joints:
- removed joint 1_5
- removed joint 2_3
- removed joint 3_4
- removed joint 5_6
- removed joint 6_7
- joint 0_1: origin xyz=0.1 0 1 rpy=0 0 0 -> xyz=-0.95 0 1 rpy=0 0 0
- joint 1_2: origin xyz=1.0 0 0 rpy=0 0 0 -> xyz=-2.25 -2.0 0 rpy=0 0 0

Commit message: Added link addition mutation

File: body.urdf (robot description, URDF)
Before this commit: robot robot, 3 links, 2 joints
Links:
- added link 3, mass 1; collision box size=1.0 2.0 4.0; visual box size=1.0 2.0 4.0
- added link 4, mass 1; collision box size=0.5 3.0 2.0; visual box size=0.5 3.0 2.0
- link 0: geometry collision box size=0.5 0.2 0.6; visual box size=0.5 0.2 0.6
- link 1: geometry collision box size=1.5 2.0 2.5; visual box size=1.5 2.0 2.5
- link 2: geometry collision box size=2.5 0.5 1.5; visual box size=2.5 0.5 1.5
Joints:
- added joint 2_3: type revolute, parent 2, child 3, origin xyz=2.5 0 0 rpy=0 0 0, axis 1 1 0, limit lower=-3.14159 upper=3.14159 effort=0.0 velocity=0.0
- added joint 3_4: type revolute, parent 3, child 4, origin xyz=1.0 0 0 rpy=0 0 0, axis 1 1 0, limit lower=-3.14159 upper=3.14159 effort=0.0 velocity=0.0
- joint 0_1: origin xyz=-0.95 0 1 rpy=0 0 0 -> xyz=0 -0.1 1 rpy=0 0 0
- joint 1_2: origin xyz=-2.25 -2.0 0 rpy=0 0 0 -> xyz=0.75 -1.0 0 rpy=0 0 0

Commit message: Added removal of links at the end of each branch, now updating weights size according to number of links

File: body.urdf (robot description, URDF)
Before this commit: robot robot, 5 links, 4 joints
Links:
- added link 5, mass 1; collision box size=3.5 2.0 4.0; visual box size=3.5 2.0 4.0
- added link 6, mass 1; collision box size=1.0 4.0 2.0; visual box size=1.0 4.0 2.0
- added link 7, mass 1; collision box size=2.5 4.0 2.0; visual box size=2.5 4.0 2.0
- link 0: geometry collision box size=0.1 1.7 1.0; visual box size=0.1 1.7 1.0
- link 1: geometry collision box size=0.5 1.5 2.5; visual box size=0.5 1.5 2.5
- link 2: geometry collision box size=4.0 2.5 3.5; visual box size=4.0 2.5 3.5
- link 3: geometry collision box size=2.0 1.0 1.5; visual box size=2.0 1.0 1.5
- link 4: geometry collision box size=4.0 4.5 1.0; visual box size=4.0 4.5 1.0
Joints:
- added joint 4_5: type revolute, parent 4, child 5, origin xyz=-4.0 0 0 rpy=0 0 0, axis 1 1 0, limit lower=-3.14159 upper=3.14159 effort=0.0 velocity=0.0
- added joint 5_6: type revolute, parent 5, child 6, origin xyz=-3.5 0 0 rpy=0 0 0, axis 1 1 0, limit lower=-3.14159 upper=3.14159 effort=0.0 velocity=0.0
- added joint 6_7: type revolute, parent 6, child 7, origin xyz=-1.0 0 0 rpy=0 0 0, axis 1 1 0, limit lower=-3.14159 upper=3.14159 effort=0.0 velocity=0.0
- joint 0_1: origin xyz=0 -0.1 1 rpy=0 0 0 -> xyz=-0.05 0 1 rpy=0 0 0
- joint 1_2: origin xyz=0.75 -1.0 0 rpy=0 0 0 -> xyz=-0.5 0 0 rpy=0 0 0
- joint 2_3: origin xyz=2.5 0 0 rpy=0 0 0 -> xyz=-4.0 0 0 rpy=0 0 0
- joint 3_4: origin xyz=1.0 0 0 rpy=0 0 0 -> xyz=-2.0 0 0 rpy=0 0 0

Commit message: Messing with weights

File: body.urdf (robot description, URDF)
Before this commit: robot robot, 8 links, 7 joints
Links:
- removed link 7
- link 0: geometry collision box size=0.8 1.5 0.7; visual box size=0.8 1.5 0.7
- link 1: geometry collision box size=4.5 3.5 4.0; visual box size=4.5 3.5 4.0
- link 2: geometry collision box size=3.0 3.5 4.5; visual box size=3.0 3.5 4.5
- link 3: geometry collision box size=0.5 3.0 3.5; visual box size=0.5 3.0 3.5
- link 4: geometry collision box size=4.5 3.0 2.0; visual box size=4.5 3.0 2.0
- link 5: geometry collision box size=4.5 3.0 3.5; visual box size=4.5 3.0 3.5
- link 6: geometry collision box size=3.0 4.5 1.0; visual box size=3.0 4.5 1.0
Joints:
- removed joint 6_7
- joint 0_1: origin xyz=-0.05 0 1 rpy=0 0 0 -> xyz=0.4 0 1 rpy=0 0 0
- joint 1_2: origin xyz=-0.5 0 0 rpy=0 0 0 -> xyz=4.5 0 0 rpy=0 0 0
- joint 2_3: origin xyz=-4.0 0 0 rpy=0 0 0 -> xyz=1.5 1.75 0 rpy=0 0 0
- joint 3_4: origin xyz=-2.0 0 0 rpy=0 0 0 -> xyz=0 3.0 0 rpy=0 0 0
- joint 4_5: origin xyz=-4.0 0 0 rpy=0 0 0 -> xyz=0 3.0 0 rpy=0 0 0
- joint 5_6: origin xyz=-3.5 0 0 rpy=0 0 0 -> xyz=0 3.0 0 rpy=0 0 0

Commit message: Working evolution with adding links. Brains evolving and functioning

File: body.urdf (robot description, URDF)
Before this commit: robot robot, 7 links, 6 joints
Links:
- link 0: geometry collision box size=1.8 0.9 0.1; visual box size=1.8 0.9 0.1
- link 1: geometry collision box size=1.5 1.0 2.5; visual box size=1.5 1.0 2.5
- link 2: geometry collision box size=4.5 3.5 4.0; visual box size=4.5 3.5 4.0
- link 3: geometry collision box size=3.5 4.0 2.0; visual box size=3.5 4.0 2.0
- link 4: geometry collision box size=3.5 1.5 4.5; visual box size=3.5 1.5 4.5
- link 5: geometry collision box size=1.5 0.5 4.5; visual box size=1.5 0.5 4.5
- link 6: geometry collision box size=1.5 4.0 2.5; visual box size=1.5 4.0 2.5
Joints:
- removed joint 4_5
- added joint 2_5: type revolute, parent 2, child 5, origin xyz=0 0 4.0 rpy=0 0 0, axis 1 1 0, limit lower=-3.14159 upper=3.14159 effort=0.0 velocity=0.0
- joint 0_1: origin xyz=0.4 0 1 rpy=0 0 0 -> xyz=0 0.45 1 rpy=0 0 0
- joint 1_2: origin xyz=4.5 0 0 rpy=0 0 0 -> xyz=0 0.5 1.25 rpy=0 0 0
- joint 2_3: origin xyz=1.5 1.75 0 rpy=0 0 0 -> xyz=0 1.75 2.0 rpy=0 0 0
- joint 3_4: origin xyz=0 3.0 0 rpy=0 0 0 -> xyz=0 4.0 0 rpy=0 0 0
- joint 5_6: origin xyz=0 3.0 0 rpy=0 0 0 -> xyz=0 0 4.5 rpy=0 0 0

Commit message: Added mutations to add or remove sensors from links

File: body.urdf (robot description, URDF)
Before this commit: robot robot, 7 links, 6 joints
Links:
- removed link 6
- added link 10, mass 1; collision box size=4 3 3; visual box size=4 3 3
- added link 7, mass 1; collision box size=1 4 4; visual box size=1 4 4
- added link 8, mass 1; collision box size=4 4 2; visual box size=4 4 2
- added link 9, mass 1; collision box size=1 2 3; visual box size=1 2 3
- link 0: geometry collision box size=1.4 0.2 1.0; visual box size=1.4 0.2 1.0
- link 1: geometry collision box size=4 1 3; visual box size=4 1 3
- link 2: geometry collision box size=3 3 4; visual box size=3 3 4
- link 3: geometry collision box size=1 1 3; visual box size=1 1 3
- link 4: geometry collision box size=2 1 2; visual box size=2 1 2
- link 5: geometry collision box size=3 1 1; visual box size=3 1 1
Joints:
- removed joint 5_6
- added joint 2_7: type revolute, parent 2, child 7, origin xyz=-3.0 0 0 rpy=0 0 0, axis 1 1 0, limit lower=-3.14159 upper=3.14159 effort=0.0 velocity=0.0
- added joint 7_8: type revolute, parent 7, child 8, origin xyz=-1.0 0 0 rpy=0 0 0, axis 1 1 0, limit lower=-3.14159 upper=3.14159 effort=0.0 velocity=0.0
- added joint 8_9: type revolute, parent 8, child 9, origin xyz=-4.0 0 0 rpy=0 0 0, axis 1 1 0, limit lower=-3.14159 upper=3.14159 effort=0.0 velocity=0.0
- added joint 9_10: type revolute, parent 9, child 10, origin xyz=-1.0 0 0 rpy=0 0 0, axis 1 1 0, limit lower=-3.14159 upper=3.14159 effort=0.0 velocity=0.0
- joint 0_1: origin xyz=0 0.45 1 rpy=0 0 0 -> xyz=0 -0.1 1 rpy=0 0 0
- joint 1_2: origin xyz=0 0.5 1.25 rpy=0 0 0 -> xyz=-2.0 -0.5 0 rpy=0 0 0
- joint 2_3: origin xyz=0 1.75 2.0 rpy=0 0 0 -> xyz=-1.5 -1.5 0 rpy=0 0 0
- joint 2_5: origin xyz=0 0 4.0 rpy=0 0 0 -> xyz=-1.5 0 2.0 rpy=0 0 0
- joint 3_4: origin xyz=0 4.0 0 rpy=0 0 0 -> xyz=0 -1.0 0 rpy=0 0 0
