Commit message: Fixed hidden neuron mutation

File: body4.urdf (robot description, URDF)
Before this commit: robot robot, 8 links, 7 joints
Links:
- added link 10, mass 1; collision box size=3 2 1; visual box size=3 2 1
- added link 8, mass 1; collision box size=2 1 2; visual box size=2 1 2
- added link 9, mass 1; collision box size=4 1 2; visual box size=4 1 2
- link 0: geometry collision box size=0.6 0.1 1.5; visual box size=0.6 0.1 1.5
- link 1: geometry collision box size=2 3 3; visual box size=2 3 3
- link 2: geometry collision box size=2 3 4; visual box size=2 3 4
- link 3: geometry collision box size=1 3 1; visual box size=1 3 1
- link 4: geometry collision box size=1 2 4; visual box size=1 2 4
- link 5: geometry collision box size=3 3 3; visual box size=3 3 3
- link 6: geometry collision box size=1 4 4; visual box size=1 4 4
- link 7: geometry collision box size=2 2 2; visual box size=2 2 2
Joints:
- added joint 1_8: type revolute, parent 1, child 8, origin xyz=0 0 3.0 rpy=0 0 0, axis 1 1 0, limit lower=-3.14159 upper=3.14159 effort=0.0 velocity=0.0
- added joint 8_9: type revolute, parent 8, child 9, origin xyz=0 0 2.0 rpy=0 0 0, axis 1 1 0, limit lower=-3.14159 upper=3.14159 effort=0.0 velocity=0.0
- added joint 9_10: type revolute, parent 9, child 10, origin xyz=0 0 2.0 rpy=0 0 0, axis 1 1 0, limit lower=-3.14159 upper=3.14159 effort=0.0 velocity=0.0
- joint 0_1: origin xyz=-0.5 0 1 rpy=0 0 0 -> xyz=0 0 1.75 rpy=0 0 0
- joint 1_2: origin xyz=-1.0 -1.0 0 rpy=0 0 0 -> xyz=0 -1.5 1.5 rpy=0 0 0
- joint 1_5: origin xyz=-1.0 1.0 0 rpy=0 0 0 -> xyz=1.0 0 1.5 rpy=0 0 0
- joint 2_3: origin xyz=0 -1.0 0 rpy=0 0 0 -> xyz=0 -3.0 0 rpy=0 0 0
- joint 3_4: origin xyz=-1.0 -1.0 0 rpy=0 0 0 -> xyz=0 -3.0 0 rpy=0 0 0
- joint 5_6: origin xyz=0 4.0 0 rpy=0 0 0 -> xyz=3.0 0 0 rpy=0 0 0
- joint 6_7: origin xyz=0 1.0 0 rpy=0 0 0 -> xyz=1.0 0 0 rpy=0 0 0
